File: DC-HVDC ConverterV2.kicad_sch (KiCad schematic)
At the start: 29 parts, among them J1 Schraubklemme, J2 Conn_01x02_Pin, J3 4er Pinreihe, J4 5er Buchsenleiste, Q1 IRF740, U3 TL3843P, U4 SKM10A-12

Commit message: ab hier mit neuem DC-DC Isolator
Parts:
- removed U4: SKM10A-12, SKM10A_MWU, symbol MEAN WELL SKM10A-12:SKM10A-12
- added U1: (no value), Eigene:DKB3-12S2PH3, symbol EigeneSymbole:DKB3-12S2PH3
- R7: footprint Resistor_SMD:R_2512_6332Metric -> Resistor_THT:R_Bare_Metal_Element_L12.4mm_W4.8mm_P11.40mm
Connections:
- net +12V: now also U1.1 (+Vin)
- net +12V_FLOATING: now also U1.5 (+Vout)
- net GND: now also U1.2 (-Vin)
- net GND_FLOATING: now also U1.7 (-Vout)
Other:
- note added: "12V 250mA galvanisch getrennt"
- note removed: "12V 800mA galvanisch getrennt"
- moved on the sheet: C7, R7
